File: PCB/MXR Distortion/MXR Distortion.kicad_pcb (KiCad board)
At the start: 2 copper layers, 117 x 54 mm, 21 parts, among them J1 AudioJack2, J2 AudioJack2, J3 Barrel_Jack_MountingPin, U1 LM741

Commit message: Added PCB, SERIE
Parts:
- added C1: 1n, Capacitor_THT:C_Disc_D3.0mm_W2.0mm_P2.50mm, F.Cu at (181.0, 43.2)
- added C1: 1n, Capacitor_THT:C_Disc_D3.0mm_W2.0mm_P2.50mm, F.Cu at (52.5, 172.5)
- added C1: 1n, Capacitor_THT:C_Disc_D3.0mm_W2.0mm_P2.50mm, F.Cu at (181.0, 111.1)
- added C1: 1n, Capacitor_THT:C_Disc_D3.0mm_W2.0mm_P2.50mm, F.Cu at (182.0, 172.5)
- added C1: 1n, Capacitor_THT:C_Disc_D3.0mm_W2.0mm_P2.50mm, F.Cu at (52.0, 110.5)
- added C2: 10n, Capacitor_THT:C_Disc_D5.0mm_W2.5mm_P5.00mm, F.Cu at (181.0, 98.4)
- added C2: 10n, Capacitor_THT:C_Disc_D5.0mm_W2.5mm_P5.00mm, F.Cu at (52.5, 159.8)
- added C2: 10n, Capacitor_THT:C_Disc_D5.0mm_W2.5mm_P5.00mm, F.Cu at (182.0, 159.8)
- added C2: 10n, Capacitor_THT:C_Disc_D5.0mm_W2.5mm_P5.00mm, F.Cu at (52.0, 97.8)
- added C2: 10n, Capacitor_THT:C_Disc_D5.0mm_W2.5mm_P5.00mm, F.Cu at (181.0, 30.5)
- added C3: 47n, Capacitor_THT:C_Radial_D6.3mm_H7.0mm_P2.50mm, F.Cu at (187.5, 110.9)
- added C3: 47n, Capacitor_THT:C_Radial_D6.3mm_H7.0mm_P2.50mm, F.Cu at (188.5, 172.2)
- added C3: 47n, Capacitor_THT:C_Radial_D6.3mm_H7.0mm_P2.50mm, F.Cu at (187.5, 43.0)
- added C3: 47n, Capacitor_THT:C_Radial_D6.3mm_H7.0mm_P2.50mm, F.Cu at (58.5, 110.2)
- added C3: 47n, Capacitor_THT:C_Radial_D6.3mm_H7.0mm_P2.50mm, F.Cu at (59.0, 172.2)
- added C4: 1u, Capacitor_THT:CP_Radial_D5.0mm_P2.00mm, F.Cu at (85.5, 89.2)
- added C4: 1u, Capacitor_THT:CP_Radial_D5.0mm_P2.00mm, F.Cu at (214.5, 89.9)
- added C4: 1u, Capacitor_THT:CP_Radial_D5.0mm_P2.00mm, F.Cu at (215.5, 151.2)
- added C4: 1u, Capacitor_THT:CP_Radial_D5.0mm_P2.00mm, F.Cu at (86.0, 151.2)
- added C4: 1u, Capacitor_THT:CP_Radial_D5.0mm_P2.00mm, F.Cu at (214.5, 22.0)
- added C5: 1n, Capacitor_THT:C_Disc_D3.0mm_W2.0mm_P2.50mm, F.Cu at (231.0, 36.2)
- added C5: 1n, Capacitor_THT:C_Disc_D3.0mm_W2.0mm_P2.50mm, F.Cu at (102.5, 165.5)
- added C5: 1n, Capacitor_THT:C_Disc_D3.0mm_W2.0mm_P2.50mm, F.Cu at (232.0, 165.5)
- added C5: 1n, Capacitor_THT:C_Disc_D3.0mm_W2.0mm_P2.50mm, F.Cu at (102.0, 103.5)
- added C5: 1n, Capacitor_THT:C_Disc_D3.0mm_W2.0mm_P2.50mm, F.Cu at (231.0, 104.1)
- added C6: 1u, Capacitor_THT:CP_Radial_D5.0mm_P2.00mm, F.Cu at (88.0, 111.2)
- added C6: 1u, Capacitor_THT:CP_Radial_D5.0mm_P2.00mm, F.Cu at (88.5, 173.2)
- added C6: 1u, Capacitor_THT:CP_Radial_D5.0mm_P2.00mm, F.Cu at (217.0, 44.0)
- added C6: 1u, Capacitor_THT:CP_Radial_D5.0mm_P2.00mm, F.Cu at (218.0, 173.2)
- added C6: 1u, Capacitor_THT:CP_Radial_D5.0mm_P2.00mm, F.Cu at (217.0, 111.9)
- added D1: D, Diode_THT:D_DO-35_SOD27_P7.62mm_Horizontal, F.Cu at (91.5, 166.2)
- added D1: D, Diode_THT:D_DO-35_SOD27_P7.62mm_Horizontal, F.Cu at (221.0, 166.2)
- added D1: D, Diode_THT:D_DO-35_SOD27_P7.62mm_Horizontal, F.Cu at (91.0, 104.2)
- added D1: D, Diode_THT:D_DO-35_SOD27_P7.62mm_Horizontal, F.Cu at (220.0, 104.9)
- added D1: D, Diode_THT:D_DO-35_SOD27_P7.62mm_Horizontal, F.Cu at (220.0, 37.0)
- added D2: D, Diode_THT:D_DO-35_SOD27_P7.62mm_Horizontal, F.Cu at (97.0, 96.4)
- added D2: D, Diode_THT:D_DO-35_SOD27_P7.62mm_Horizontal, F.Cu at (226.0, 97.1)
- added D2: D, Diode_THT:D_DO-35_SOD27_P7.62mm_Horizontal, F.Cu at (97.5, 158.4)
- added D2: D, Diode_THT:D_DO-35_SOD27_P7.62mm_Horizontal, F.Cu at (227.0, 158.4)
- added D2: D, Diode_THT:D_DO-35_SOD27_P7.62mm_Horizontal, F.Cu at (226.0, 29.2)
- added J1: AudioJack2, Connector_Audio:Jack_6.35mm_Neutrik_NMJ4HCD2_Horizontal, F.Cu at (170.5, 114.9)
- added J1: AudioJack2, Connector_Audio:Jack_6.35mm_Neutrik_NMJ4HCD2_Horizontal, F.Cu at (42.0, 176.2)
- added J1: AudioJack2, Connector_Audio:Jack_6.35mm_Neutrik_NMJ4HCD2_Horizontal, F.Cu at (41.5, 114.2)
- added J1: AudioJack2, Connector_Audio:Jack_6.35mm_Neutrik_NMJ4HCD2_Horizontal, F.Cu at (170.5, 47.0)
- added J1: AudioJack2, Connector_Audio:Jack_6.35mm_Neutrik_NMJ4HCD2_Horizontal, F.Cu at (171.5, 176.2)
- added J2: AudioJack2, Connector_Audio:Jack_6.35mm_Neutrik_NMJ4HCD2_Horizontal, F.Cu at (112.1, 98.1)
- added J2: AudioJack2, Connector_Audio:Jack_6.35mm_Neutrik_NMJ4HCD2_Horizontal, F.Cu at (241.1, 30.9)
- added J2: AudioJack2, Connector_Audio:Jack_6.35mm_Neutrik_NMJ4HCD2_Horizontal, F.Cu at (112.6, 160.1)
- added J2: AudioJack2, Connector_Audio:Jack_6.35mm_Neutrik_NMJ4HCD2_Horizontal, F.Cu at (241.1, 98.8)
- added J2: AudioJack2, Connector_Audio:Jack_6.35mm_Neutrik_NMJ4HCD2_Horizontal, F.Cu at (242.1, 160.1)
- added J3: Barrel_Jack_MountingPin, Connector_BarrelJack:BarrelJack_Horizontal, F.Cu at (75.8, 120.8)
- added J3: Barrel_Jack_MountingPin, Connector_BarrelJack:BarrelJack_Horizontal, F.Cu at (76.3, 182.8)
- added J3: Barrel_Jack_MountingPin, Connector_BarrelJack:BarrelJack_Horizontal, F.Cu at (205.8, 182.8)
- added J3: Barrel_Jack_MountingPin, Connector_BarrelJack:BarrelJack_Horizontal, F.Cu at (204.8, 53.5)
- added J3: Barrel_Jack_MountingPin, Connector_BarrelJack:BarrelJack_Horizontal, F.Cu at (204.8, 121.4)
- added R1: 10K, Resistor_THT:R_Axial_DIN0207_L6.3mm_D2.5mm_P7.62mm_Horizontal, F.Cu at (183.2, 155.8)
- added R1: 10K, Resistor_THT:R_Axial_DIN0207_L6.3mm_D2.5mm_P7.62mm_Horizontal, F.Cu at (182.2, 94.4)
- added R1: 10K, Resistor_THT:R_Axial_DIN0207_L6.3mm_D2.5mm_P7.62mm_Horizontal, F.Cu at (53.2, 93.8)
- added R1: 10K, Resistor_THT:R_Axial_DIN0207_L6.3mm_D2.5mm_P7.62mm_Horizontal, F.Cu at (182.2, 26.5)
- added R1: 10K, Resistor_THT:R_Axial_DIN0207_L6.3mm_D2.5mm_P7.62mm_Horizontal, F.Cu at (53.7, 155.8)
- added R2: 1M, Resistor_THT:R_Axial_DIN0207_L6.3mm_D2.5mm_P7.62mm_Horizontal, F.Cu at (62.0, 104.6)
- added R2: 1M, Resistor_THT:R_Axial_DIN0207_L6.3mm_D2.5mm_P7.62mm_Horizontal, F.Cu at (62.5, 166.6)
- added R2: 1M, Resistor_THT:R_Axial_DIN0207_L6.3mm_D2.5mm_P7.62mm_Horizontal, F.Cu at (191.0, 105.2)
- added R2: 1M, Resistor_THT:R_Axial_DIN0207_L6.3mm_D2.5mm_P7.62mm_Horizontal, F.Cu at (192.0, 166.6)
- added R2: 1M, Resistor_THT:R_Axial_DIN0207_L6.3mm_D2.5mm_P7.62mm_Horizontal, F.Cu at (191.0, 37.3)
- added R3: 4.7K, Resistor_THT:R_Axial_DIN0207_L6.3mm_D2.5mm_P7.62mm_Horizontal, F.Cu at (194.5, 47.5)
- added R3: 4.7K, Resistor_THT:R_Axial_DIN0207_L6.3mm_D2.5mm_P7.62mm_Horizontal, F.Cu at (194.5, 115.4)
- added R3: 4.7K, Resistor_THT:R_Axial_DIN0207_L6.3mm_D2.5mm_P7.62mm_Horizontal, F.Cu at (195.5, 176.8)
- added R3: 4.7K, Resistor_THT:R_Axial_DIN0207_L6.3mm_D2.5mm_P7.62mm_Horizontal, F.Cu at (65.5, 114.8)
- added R3: 4.7K, Resistor_THT:R_Axial_DIN0207_L6.3mm_D2.5mm_P7.62mm_Horizontal, F.Cu at (66.0, 176.8)
- added R4: 1M, Resistor_THT:R_Axial_DIN0207_L6.3mm_D2.5mm_P7.62mm_Horizontal, F.Cu at (202.2, 149.8)
- added R4: 1M, Resistor_THT:R_Axial_DIN0207_L6.3mm_D2.5mm_P7.62mm_Horizontal, F.Cu at (201.2, 20.5)
- added R4: 1M, Resistor_THT:R_Axial_DIN0207_L6.3mm_D2.5mm_P7.62mm_Horizontal, F.Cu at (201.2, 88.4)
- added R4: 1M, Resistor_THT:R_Axial_DIN0207_L6.3mm_D2.5mm_P7.62mm_Horizontal, F.Cu at (72.2, 87.8)
- added R4: 1M, Resistor_THT:R_Axial_DIN0207_L6.3mm_D2.5mm_P7.62mm_Horizontal, F.Cu at (72.7, 149.8)
- added R5: 10K, Resistor_THT:R_Axial_DIN0207_L6.3mm_D2.5mm_P7.62mm_Horizontal, F.Cu at (85.0, 158.4)
- added R5: 10K, Resistor_THT:R_Axial_DIN0207_L6.3mm_D2.5mm_P7.62mm_Horizontal, F.Cu at (213.5, 29.2)
- added R5: 10K, Resistor_THT:R_Axial_DIN0207_L6.3mm_D2.5mm_P7.62mm_Horizontal, F.Cu at (214.5, 158.4)
- added R5: 10K, Resistor_THT:R_Axial_DIN0207_L6.3mm_D2.5mm_P7.62mm_Horizontal, F.Cu at (213.5, 97.1)
- added R5: 10K, Resistor_THT:R_Axial_DIN0207_L6.3mm_D2.5mm_P7.62mm_Horizontal, F.Cu at (84.5, 96.4)
- added R6: 1M, Resistor_THT:R_Axial_DIN0207_L6.3mm_D2.5mm_P7.62mm_Horizontal, F.Cu at (204.9, 173.2)
- added R6: 1M, Resistor_THT:R_Axial_DIN0207_L6.3mm_D2.5mm_P7.62mm_Horizontal, F.Cu at (203.9, 111.9)
- added R6: 1M, Resistor_THT:R_Axial_DIN0207_L6.3mm_D2.5mm_P7.62mm_Horizontal, F.Cu at (74.9, 111.2)
- added R6: 1M, Resistor_THT:R_Axial_DIN0207_L6.3mm_D2.5mm_P7.62mm_Horizontal, F.Cu at (203.9, 44.0)
- added R6: 1M, Resistor_THT:R_Axial_DIN0207_L6.3mm_D2.5mm_P7.62mm_Horizontal, F.Cu at (75.4, 173.2)
- added R7: 1M, Resistor_THT:R_Axial_DIN0207_L6.3mm_D2.5mm_P7.62mm_Horizontal, F.Cu at (64.0, 111.2)
- added R7: 1M, Resistor_THT:R_Axial_DIN0207_L6.3mm_D2.5mm_P7.62mm_Horizontal, F.Cu at (194.0, 173.2)
- added R7: 1M, Resistor_THT:R_Axial_DIN0207_L6.3mm_D2.5mm_P7.62mm_Horizontal, F.Cu at (193.0, 111.9)
- added R7: 1M, Resistor_THT:R_Axial_DIN0207_L6.3mm_D2.5mm_P7.62mm_Horizontal, F.Cu at (193.0, 44.0)
- added R7: 1M, Resistor_THT:R_Axial_DIN0207_L6.3mm_D2.5mm_P7.62mm_Horizontal, F.Cu at (64.5, 173.2)
- added RV1: 10K, Potentiometer_THT:Potentiometer_Alps_RK163_Single_Horizontal, F.Cu at (220.0, 185.7)
- added RV1: 10K, Potentiometer_THT:Potentiometer_Alps_RK163_Single_Horizontal, F.Cu at (90.0, 123.7)
- added RV1: 10K, Potentiometer_THT:Potentiometer_Alps_RK163_Single_Horizontal, F.Cu at (219.0, 56.5)
- added RV1: 10K, Potentiometer_THT:Potentiometer_Alps_RK163_Single_Horizontal, F.Cu at (90.5, 185.7)
- added RV1: 10K, Potentiometer_THT:Potentiometer_Alps_RK163_Single_Horizontal, F.Cu at (219.0, 124.3)
- added RV2: 1M, Potentiometer_THT:Potentiometer_Alps_RK163_Single_Horizontal, F.Cu at (182.5, 56.5)
- added RV2: 1M, Potentiometer_THT:Potentiometer_Alps_RK163_Single_Horizontal, F.Cu at (182.5, 124.3)
- added RV2: 1M, Potentiometer_THT:Potentiometer_Alps_RK163_Single_Horizontal, F.Cu at (53.5, 123.7)
- added RV2: 1M, Potentiometer_THT:Potentiometer_Alps_RK163_Single_Horizontal, F.Cu at (183.5, 185.7)
- added RV2: 1M, Potentiometer_THT:Potentiometer_Alps_RK163_Single_Horizontal, F.Cu at (54.0, 185.7)
- added U1: LM741, Package_DIP:DIP-8_W7.62mm, F.Cu at (198.4, 28.9)
- added U1: LM741, Package_DIP:DIP-8_W7.62mm, F.Cu at (69.4, 96.1)
- added U1: LM741, Package_DIP:DIP-8_W7.62mm, F.Cu at (198.4, 96.8)
- added U1: LM741, Package_DIP:DIP-8_W7.62mm, F.Cu at (199.4, 158.1)
- added U1: LM741, Package_DIP:DIP-8_W7.62mm, F.Cu at (69.9, 158.1)
- moved J2 68.4 mm to (111.7, 31.3)
- moved J3 68.4 mm to (75.4, 53.9)
- moved C1 68.4 mm to (51.6, 43.6)
- moved C2 68.4 mm to (51.6, 30.9)
- moved C3 68.4 mm to (58.1, 43.4)
- moved C4 68.4 mm to (85.1, 22.4)
- moved C5 68.4 mm to (101.6, 36.6)
- moved C6 68.4 mm to (87.6, 44.4)
- moved D1 68.4 mm to (90.6, 37.4)
- moved D2 68.4 mm to (96.6, 29.6)
- moved J1 68.4 mm to (41.1, 47.4)
- moved R1 68.4 mm to (52.8, 26.9)
- moved R2 68.4 mm to (61.6, 37.7)
- moved R3 68.4 mm to (65.1, 47.9)
- moved R4 68.4 mm to (71.8, 20.9)
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Routing:
- net +9v: track 53.9 -> 323.5 mm
- net Net-(J2-PadS): track 53.0 -> 317.8 mm
- net Net-(U1--): track 43.8 -> 263.1 mm
- net Net-(D1-K): track 40.5 -> 242.9 mm
- net Net-(C1-Pad2): track 34.1 -> 204.9 mm
- net Net-(C4-Pad2): track 19.5 -> 117.1 mm
- net +4.5v: track 18.5 -> 110.7 mm
- net Net-(U1-+): track 12.8 -> 77.0 mm
- net Net-(C3-Pad2): track 9.79 -> 58.8 mm
- net Net-(R3-Pad1): track 8.52 -> 51.1 mm
- net Net-(C4-Pad1): track 7.60 -> 45.6 mm
- net Net-(C2-Pad1): track 4.49 -> 27.0 mm
- net GND: track 0.71 -> 4.25 mm
Other:
- board size 117 x 54 mm -> 245.4 x 182.8 mm

Commit message: Simulation
Parts:
- removed the C1 at (181.0, 43.2)
- removed the C1 at (52.5, 172.5)
- removed the C1 at (181.0, 111.1)
- removed the C1 at (182.0, 172.5)
- removed the C1 at (52.0, 110.5)
- removed the C2 at (181.0, 98.4)
- removed the C2 at (52.5, 159.8)
- removed the C2 at (182.0, 159.8)
- removed the C2 at (52.0, 97.8)
- removed the C2 at (181.0, 30.5)
- removed the C3 at (187.5, 110.9)
- removed the C3 at (188.5, 172.2)
- removed the C3 at (187.5, 43.0)
- removed the C3 at (58.5, 110.2)
- removed the C3 at (59.0, 172.2)
- removed the C4 at (85.5, 89.2)
- removed the C4 at (214.5, 89.9)
- removed the C4 at (215.5, 151.2)
- removed the C4 at (86.0, 151.2)
- removed the C4 at (214.5, 22.0)
- removed the C5 at (231.0, 36.2)
- removed the C5 at (102.5, 165.5)
- removed the C5 at (232.0, 165.5)
- removed the C5 at (102.0, 103.5)
- removed the C5 at (231.0, 104.1)
- removed the C6 at (88.0, 111.2)
- removed the C6 at (88.5, 173.2)
- removed the C6 at (217.0, 44.0)
- removed the C6 at (218.0, 173.2)
- removed the C6 at (217.0, 111.9)
- removed the D1 at (91.5, 166.2)
- removed the D1 at (221.0, 166.2)
- removed the D1 at (91.0, 104.2)
- removed the D1 at (220.0, 104.9)
- removed the D1 at (220.0, 37.0)
- removed the D2 at (97.0, 96.4)
- removed the D2 at (226.0, 97.1)
- removed the D2 at (97.5, 158.4)
- removed the D2 at (227.0, 158.4)
- removed the D2 at (226.0, 29.2)
- removed the J1 at (170.5, 114.9)
- removed the J1 at (42.0, 176.2)
- removed the J1 at (41.5, 114.2)
- removed the J1 at (170.5, 47.0)
- removed the J1 at (171.5, 176.2)
- removed the J2 at (112.1, 98.1)
- removed the J2 at (241.1, 30.9)
- removed the J2 at (112.6, 160.1)
- removed the J2 at (241.1, 98.8)
- removed the J2 at (242.1, 160.1)
- removed the J3 at (75.8, 120.8)
- removed the J3 at (76.3, 182.8)
- removed the J3 at (205.8, 182.8)
- removed the J3 at (204.8, 53.5)
- removed the J3 at (204.8, 121.4)
- removed the R1 at (183.2, 155.8)
- removed the R1 at (182.2, 94.4)
- removed the R1 at (53.2, 93.8)
- removed the R1 at (182.2, 26.5)
- removed the R1 at (53.7, 155.8)
- removed the R2 at (62.0, 104.6)
- removed the R2 at (62.5, 166.6)
- removed the R2 at (191.0, 105.2)
- removed the R2 at (192.0, 166.6)
- removed the R2 at (191.0, 37.3)
- removed the R3 at (194.5, 47.5)
- removed the R3 at (194.5, 115.4)
- removed the R3 at (195.5, 176.8)
- removed the R3 at (65.5, 114.8)
- removed the R3 at (66.0, 176.8)
- removed the R4 at (202.2, 149.8)
- removed the R4 at (201.2, 20.5)
- removed the R4 at (201.2, 88.4)
- removed the R4 at (72.2, 87.8)
- removed the R4 at (72.7, 149.8)
- removed the R5 at (85.0, 158.4)
- removed the R5 at (213.5, 29.2)
- removed the R5 at (214.5, 158.4)
- removed the R5 at (213.5, 97.1)
- removed the R5 at (84.5, 96.4)
- removed the R6 at (204.9, 173.2)
- removed the R6 at (203.9, 111.9)
- removed the R6 at (74.9, 111.2)
- removed the R6 at (203.9, 44.0)
- removed the R6 at (75.4, 173.2)
- removed the R7 at (64.0, 111.2)
- removed the R7 at (194.0, 173.2)
- removed the R7 at (193.0, 111.9)
- removed the R7 at (193.0, 44.0)
- removed the R7 at (64.5, 173.2)
- removed the RV1 at (220.0, 185.7)
- removed the RV1 at (90.0, 123.7)
- removed the RV1 at (219.0, 56.5)
- removed the RV1 at (90.5, 185.7)
- removed the RV1 at (219.0, 124.3)
- removed the RV2 at (182.5, 56.5)
- removed the RV2 at (182.5, 124.3)
- removed the RV2 at (53.5, 123.7)
- removed the RV2 at (183.5, 185.7)
- removed the RV2 at (54.0, 185.7)
- removed the U1 at (198.4, 28.9)
- removed the U1 at (69.4, 96.1)
- removed the U1 at (198.4, 96.8)
- removed the U1 at (199.4, 158.1)
- removed the U1 at (69.9, 158.1)
- added C1: 1n, Capacitor_THT:C_Disc_D3.0mm_W2.0mm_P2.50mm, F.Cu at (52.0, 106.8)
- added C1: 1n, Capacitor_THT:C_Disc_D3.0mm_W2.0mm_P2.50mm, F.Cu at (183.5, 43.8)
- added C1: 1n, Capacitor_THT:C_Disc_D3.0mm_W2.0mm_P2.50mm, F.Cu at (184.5, 169.8)
- added C1: 1n, Capacitor_THT:C_Disc_D3.0mm_W2.0mm_P2.50mm, F.Cu at (52.5, 170.8)
- added C1: 1n, Capacitor_THT:C_Disc_D3.0mm_W2.0mm_P2.50mm, F.Cu at (184.0, 106.2)
- added C2: 10n, Capacitor_THT:C_Disc_D5.0mm_W2.5mm_P5.00mm, F.Cu at (52.5, 158.0)
- added C2: 10n, Capacitor_THT:C_Disc_D5.0mm_W2.5mm_P5.00mm, F.Cu at (184.5, 157.0)
- added C2: 10n, Capacitor_THT:C_Disc_D5.0mm_W2.5mm_P5.00mm, F.Cu at (183.5, 31.0)
- added C2: 10n, Capacitor_THT:C_Disc_D5.0mm_W2.5mm_P5.00mm, F.Cu at (184.0, 93.5)
- added C2: 10n, Capacitor_THT:C_Disc_D5.0mm_W2.5mm_P5.00mm, F.Cu at (52.0, 94.0)
- added C3: 47n, Capacitor_THT:C_Radial_D6.3mm_H7.0mm_P2.50mm, F.Cu at (59.0, 170.5)
- added C3: 47n, Capacitor_THT:C_Radial_D6.3mm_H7.0mm_P2.50mm, F.Cu at (191.0, 169.5)
- added C3: 47n, Capacitor_THT:C_Radial_D6.3mm_H7.0mm_P2.50mm, F.Cu at (190.0, 43.5)
- added C3: 47n, Capacitor_THT:C_Radial_D6.3mm_H7.0mm_P2.50mm, F.Cu at (190.5, 106.0)
- added C3: 47n, Capacitor_THT:C_Radial_D6.3mm_H7.0mm_P2.50mm, F.Cu at (58.5, 106.5)
- added C4: 1u, Capacitor_THT:CP_Radial_D5.0mm_P2.00mm, F.Cu at (217.0, 22.5)
- added C4: 1u, Capacitor_THT:CP_Radial_D5.0mm_P2.00mm, F.Cu at (85.5, 85.5)
- added C4: 1u, Capacitor_THT:CP_Radial_D5.0mm_P2.00mm, F.Cu at (218.0, 148.5)
- added C4: 1u, Capacitor_THT:CP_Radial_D5.0mm_P2.00mm, F.Cu at (217.5, 85.0)
- added C4: 1u, Capacitor_THT:CP_Radial_D5.0mm_P2.00mm, F.Cu at (86.0, 149.5)
- added C5: 1n, Capacitor_THT:C_Disc_D3.0mm_W2.0mm_P2.50mm, F.Cu at (234.5, 162.8)
- added C5: 1n, Capacitor_THT:C_Disc_D3.0mm_W2.0mm_P2.50mm, F.Cu at (102.0, 99.8)
- added C5: 1n, Capacitor_THT:C_Disc_D3.0mm_W2.0mm_P2.50mm, F.Cu at (234.0, 99.2)
- added C5: 1n, Capacitor_THT:C_Disc_D3.0mm_W2.0mm_P2.50mm, F.Cu at (233.5, 36.8)
- added C5: 1n, Capacitor_THT:C_Disc_D3.0mm_W2.0mm_P2.50mm, F.Cu at (102.5, 163.8)
- added C6: 1u, Capacitor_THT:CP_Radial_D5.0mm_P2.00mm, F.Cu at (219.5, 44.5)
- added C6: 1u, Capacitor_THT:CP_Radial_D5.0mm_P2.00mm, F.Cu at (88.0, 107.5)
- added C6: 1u, Capacitor_THT:CP_Radial_D5.0mm_P2.00mm, F.Cu at (220.0, 107.0)
- added C6: 1u, Capacitor_THT:CP_Radial_D5.0mm_P2.00mm, F.Cu at (220.5, 170.5)
- added C6: 1u, Capacitor_THT:CP_Radial_D5.0mm_P2.00mm, F.Cu at (88.5, 171.5)
- added D1: D, Diode_THT:D_DO-35_SOD27_P7.62mm_Horizontal, F.Cu at (91.0, 100.5)
- added D1: D, Diode_THT:D_DO-35_SOD27_P7.62mm_Horizontal, F.Cu at (222.5, 37.5)
- added D1: D, Diode_THT:D_DO-35_SOD27_P7.62mm_Horizontal, F.Cu at (91.5, 164.5)
- added D1: D, Diode_THT:D_DO-35_SOD27_P7.62mm_Horizontal, F.Cu at (223.5, 163.5)
- added D1: D, Diode_THT:D_DO-35_SOD27_P7.62mm_Horizontal, F.Cu at (223.0, 100.0)
- added D2: D, Diode_THT:D_DO-35_SOD27_P7.62mm_Horizontal, F.Cu at (97.5, 156.7)
- added D2: D, Diode_THT:D_DO-35_SOD27_P7.62mm_Horizontal, F.Cu at (228.5, 29.7)
- added D2: D, Diode_THT:D_DO-35_SOD27_P7.62mm_Horizontal, F.Cu at (229.5, 155.7)
- added D2: D, Diode_THT:D_DO-35_SOD27_P7.62mm_Horizontal, F.Cu at (97.0, 92.7)
- added D2: D, Diode_THT:D_DO-35_SOD27_P7.62mm_Horizontal, F.Cu at (229.0, 92.2)
- added J1: AudioJack2, Connector_Audio:Jack_6.35mm_Neutrik_NMJ4HCD2_Horizontal, F.Cu at (41.5, 110.5)
- added J1: AudioJack2, Connector_Audio:Jack_6.35mm_Neutrik_NMJ4HCD2_Horizontal, F.Cu at (173.0, 47.5)
- added J1: AudioJack2, Connector_Audio:Jack_6.35mm_Neutrik_NMJ4HCD2_Horizontal, F.Cu at (173.5, 110.0)
- added J1: AudioJack2, Connector_Audio:Jack_6.35mm_Neutrik_NMJ4HCD2_Horizontal, F.Cu at (174.0, 173.5)
- added J1: AudioJack2, Connector_Audio:Jack_6.35mm_Neutrik_NMJ4HCD2_Horizontal, F.Cu at (42.0, 174.5)
- added J2: AudioJack2, Connector_Audio:Jack_6.35mm_Neutrik_NMJ4HCD2_Horizontal, F.Cu at (244.1, 93.9)
- added J2: AudioJack2, Connector_Audio:Jack_6.35mm_Neutrik_NMJ4HCD2_Horizontal, F.Cu at (244.6, 157.4)
- added J2: AudioJack2, Connector_Audio:Jack_6.35mm_Neutrik_NMJ4HCD2_Horizontal, F.Cu at (112.6, 158.4)
- added J2: AudioJack2, Connector_Audio:Jack_6.35mm_Neutrik_NMJ4HCD2_Horizontal, F.Cu at (112.1, 94.4)
- added J2: AudioJack2, Connector_Audio:Jack_6.35mm_Neutrik_NMJ4HCD2_Horizontal, F.Cu at (243.6, 31.4)
- added J3: Barrel_Jack_MountingPin, Connector_BarrelJack:BarrelJack_Horizontal, F.Cu at (207.3, 54.0)
- added J3: Barrel_Jack_MountingPin, Connector_BarrelJack:BarrelJack_Horizontal, F.Cu at (76.3, 181.0)
- added J3: Barrel_Jack_MountingPin, Connector_BarrelJack:BarrelJack_Horizontal, F.Cu at (208.3, 180.0)
- added J3: Barrel_Jack_MountingPin, Connector_BarrelJack:BarrelJack_Horizontal, F.Cu at (75.8, 117.0)
- added J3: Barrel_Jack_MountingPin, Connector_BarrelJack:BarrelJack_Horizontal, F.Cu at (207.8, 116.5)
- added R1: 10K, Resistor_THT:R_Axial_DIN0207_L6.3mm_D2.5mm_P7.62mm_Horizontal, F.Cu at (184.7, 27.0)
- added R1: 10K, Resistor_THT:R_Axial_DIN0207_L6.3mm_D2.5mm_P7.62mm_Horizontal, F.Cu at (53.7, 154.0)
- added R1: 10K, Resistor_THT:R_Axial_DIN0207_L6.3mm_D2.5mm_P7.62mm_Horizontal, F.Cu at (185.2, 89.5)
- added R1: 10K, Resistor_THT:R_Axial_DIN0207_L6.3mm_D2.5mm_P7.62mm_Horizontal, F.Cu at (53.2, 90.0)
- added R1: 10K, Resistor_THT:R_Axial_DIN0207_L6.3mm_D2.5mm_P7.62mm_Horizontal, F.Cu at (185.7, 153.0)
- added R2: 1M, Resistor_THT:R_Axial_DIN0207_L6.3mm_D2.5mm_P7.62mm_Horizontal, F.Cu at (194.0, 100.3)
- added R2: 1M, Resistor_THT:R_Axial_DIN0207_L6.3mm_D2.5mm_P7.62mm_Horizontal, F.Cu at (62.5, 164.8)
- added R2: 1M, Resistor_THT:R_Axial_DIN0207_L6.3mm_D2.5mm_P7.62mm_Horizontal, F.Cu at (194.5, 163.8)
- added R2: 1M, Resistor_THT:R_Axial_DIN0207_L6.3mm_D2.5mm_P7.62mm_Horizontal, F.Cu at (62.0, 100.8)
- added R2: 1M, Resistor_THT:R_Axial_DIN0207_L6.3mm_D2.5mm_P7.62mm_Horizontal, F.Cu at (193.5, 37.8)
- added R3: 4.7K, Resistor_THT:R_Axial_DIN0207_L6.3mm_D2.5mm_P7.62mm_Horizontal, F.Cu at (66.0, 175.0)
- added R3: 4.7K, Resistor_THT:R_Axial_DIN0207_L6.3mm_D2.5mm_P7.62mm_Horizontal, F.Cu at (197.0, 48.0)
- added R3: 4.7K, Resistor_THT:R_Axial_DIN0207_L6.3mm_D2.5mm_P7.62mm_Horizontal, F.Cu at (197.5, 110.5)
- added R3: 4.7K, Resistor_THT:R_Axial_DIN0207_L6.3mm_D2.5mm_P7.62mm_Horizontal, F.Cu at (65.5, 111.0)
- added R3: 4.7K, Resistor_THT:R_Axial_DIN0207_L6.3mm_D2.5mm_P7.62mm_Horizontal, F.Cu at (198.0, 174.0)
- added R4: 1M, Resistor_THT:R_Axial_DIN0207_L6.3mm_D2.5mm_P7.62mm_Horizontal, F.Cu at (204.2, 83.5)
- added R4: 1M, Resistor_THT:R_Axial_DIN0207_L6.3mm_D2.5mm_P7.62mm_Horizontal, F.Cu at (72.7, 148.0)
- added R4: 1M, Resistor_THT:R_Axial_DIN0207_L6.3mm_D2.5mm_P7.62mm_Horizontal, F.Cu at (203.7, 21.0)
- added R4: 1M, Resistor_THT:R_Axial_DIN0207_L6.3mm_D2.5mm_P7.62mm_Horizontal, F.Cu at (72.2, 84.0)
- added R4: 1M, Resistor_THT:R_Axial_DIN0207_L6.3mm_D2.5mm_P7.62mm_Horizontal, F.Cu at (204.7, 147.0)
- added R5: 10K, Resistor_THT:R_Axial_DIN0207_L6.3mm_D2.5mm_P7.62mm_Horizontal, F.Cu at (85.0, 156.7)
- added R5: 10K, Resistor_THT:R_Axial_DIN0207_L6.3mm_D2.5mm_P7.62mm_Horizontal, F.Cu at (216.5, 92.2)
- added R5: 10K, Resistor_THT:R_Axial_DIN0207_L6.3mm_D2.5mm_P7.62mm_Horizontal, F.Cu at (84.5, 92.7)
- added R5: 10K, Resistor_THT:R_Axial_DIN0207_L6.3mm_D2.5mm_P7.62mm_Horizontal, F.Cu at (216.0, 29.7)
- added R5: 10K, Resistor_THT:R_Axial_DIN0207_L6.3mm_D2.5mm_P7.62mm_Horizontal, F.Cu at (217.0, 155.7)
- added R6: 1M, Resistor_THT:R_Axial_DIN0207_L6.3mm_D2.5mm_P7.62mm_Horizontal, F.Cu at (207.4, 170.5)
- added R6: 1M, Resistor_THT:R_Axial_DIN0207_L6.3mm_D2.5mm_P7.62mm_Horizontal, F.Cu at (75.4, 171.5)
- added R6: 1M, Resistor_THT:R_Axial_DIN0207_L6.3mm_D2.5mm_P7.62mm_Horizontal, F.Cu at (74.9, 107.5)
- added R6: 1M, Resistor_THT:R_Axial_DIN0207_L6.3mm_D2.5mm_P7.62mm_Horizontal, F.Cu at (206.9, 107.0)
- added R6: 1M, Resistor_THT:R_Axial_DIN0207_L6.3mm_D2.5mm_P7.62mm_Horizontal, F.Cu at (206.4, 44.5)
- added R7: 1M, Resistor_THT:R_Axial_DIN0207_L6.3mm_D2.5mm_P7.62mm_Horizontal, F.Cu at (196.0, 107.0)
- added R7: 1M, Resistor_THT:R_Axial_DIN0207_L6.3mm_D2.5mm_P7.62mm_Horizontal, F.Cu at (64.5, 171.5)
- added R7: 1M, Resistor_THT:R_Axial_DIN0207_L6.3mm_D2.5mm_P7.62mm_Horizontal, F.Cu at (195.5, 44.5)
- added R7: 1M, Resistor_THT:R_Axial_DIN0207_L6.3mm_D2.5mm_P7.62mm_Horizontal, F.Cu at (196.5, 170.5)
- added R7: 1M, Resistor_THT:R_Axial_DIN0207_L6.3mm_D2.5mm_P7.62mm_Horizontal, F.Cu at (64.0, 107.5)
- added RV1: 10K, Potentiometer_THT:Potentiometer_Alps_RK163_Single_Horizontal, F.Cu at (221.5, 57.0)
- added RV1: 10K, Potentiometer_THT:Potentiometer_Alps_RK163_Single_Horizontal, F.Cu at (222.0, 119.5)
- added RV1: 10K, Potentiometer_THT:Potentiometer_Alps_RK163_Single_Horizontal, F.Cu at (222.5, 182.9)
- added RV1: 10K, Potentiometer_THT:Potentiometer_Alps_RK163_Single_Horizontal, F.Cu at (90.0, 120.0)
- added RV1: 10K, Potentiometer_THT:Potentiometer_Alps_RK163_Single_Horizontal, F.Cu at (90.5, 183.9)
- added RV2: 1M, Potentiometer_THT:Potentiometer_Alps_RK163_Single_Horizontal, F.Cu at (53.5, 120.0)
- added RV2: 1M, Potentiometer_THT:Potentiometer_Alps_RK163_Single_Horizontal, F.Cu at (186.0, 182.9)
- added RV2: 1M, Potentiometer_THT:Potentiometer_Alps_RK163_Single_Horizontal, F.Cu at (54.0, 183.9)
- added RV2: 1M, Potentiometer_THT:Potentiometer_Alps_RK163_Single_Horizontal, F.Cu at (185.5, 119.5)
- added RV2: 1M, Potentiometer_THT:Potentiometer_Alps_RK163_Single_Horizontal, F.Cu at (185.0, 57.0)
- added U1: LM741, Package_DIP:DIP-8_W7.62mm, F.Cu at (201.4, 91.9)
- added U1: LM741, Package_DIP:DIP-8_W7.62mm, F.Cu at (69.4, 92.4)
- added U1: LM741, Package_DIP:DIP-8_W7.62mm, F.Cu at (201.9, 155.4)
- added U1: LM741, Package_DIP:DIP-8_W7.62mm, F.Cu at (200.9, 29.4)
- added U1: LM741, Package_DIP:DIP-8_W7.62mm, F.Cu at (69.9, 156.4)
Connections:
- R2 pad 1: GND -> +4.5v
Other:
- board size 245.4 x 182.8 mm -> 247.9 x 180.6 mm
